Commit message: Changed imu inertia and <!--collision--> Changed sensor-axis inertias

File: urdf/axis.urdf.xacro (robot description, xacro)
@@ -17,6 +17,5 @@
         <origin xyz="0.0 0.0 0.0" rpy="0 0 0"/>
         <mass value="0.1"/>
-        <origin xyz="0 0 0" rpy="0 0 0"/>
-        <inertia ixx="0.1" ixy="0" ixz="0" iyy="0.1" iyz="0" izz="0.1"/>
+        <inertia ixx="0.0004008333" ixy="0" ixz="0" iyy="0.0004008333" iyz="0" izz="0.000426666"/>
       </inertial>
       <visual>
@@ -49,7 +48,7 @@
     <link name="${prefix}_pan_link">
       <inertial>
+        <origin xyz="0.0 0.0 0.0" rpy="0 0 0"/>
         <mass value="0.1"/>
-        <origin xyz="0 0 0" rpy="0 0 0"/>
-        <inertia ixx="0.1" ixy="0" ixz="0" iyy="0.1" iyz="0" izz="0.1"/>
+        <inertia ixx="0.0004008333" ixy="0" ixz="0" iyy="0.0004008333" iyz="0" izz="0.000426666"/>
       </inertial>
     </link>
@@ -74,7 +73,7 @@
     <link name="${prefix}_tilt_link">
       <inertial>
+        <origin xyz="0.0 0.0 0.0" rpy="0 0 0"/>
         <mass value="0.1"/>
-        <origin xyz="0 0 0" rpy="0 0 0"/>
-        <inertia ixx="0.1" ixy="0" ixz="0" iyy="0.1" iyz="0" izz="0.1"/>
+        <inertia ixx="0.0004008333" ixy="0" ixz="0" iyy="0.0004008333" iyz="0" izz="0.000426666"/>
       </inertial>
     </link>

File: urdf/imu.urdf.xacro (robot description, xacro)
@@ -13,5 +13,5 @@
 	        <mass value="0.001"/>
 	        <origin rpy="0 0 0" xyz="0 0 0"/>
-	        <inertia ixx="0.0001" ixy="0" ixz="0" iyy="0.000001" iyz="0" izz="0.0001"/>
+	        <inertia ixx="0.00000000167" ixy="0" ixz="0" iyy="0.00000000167" iyz="0" izz="0.00000000167"/>
 	      </inertial>
 	      <visual>
@@ -21,10 +21,10 @@
 	        </geometry>
 	      </visual>
-	      <collision>
+	      <!--collision>
 	        <origin rpy="0 0 0" xyz="0 0 0"/>
 	        <geometry>
 	          <box size=".001 .001 .001"/>
 	        </geometry>
-	      </collision>
+	      </collision-->
 	  </link>
 	  <!--<gazebo>-->
