Commit message: RS_BPearl: added bpearl before every link and joint

File: urdf/rs_bpearl.urdf.xacro (robot description, xacro)
@@ -6,10 +6,10 @@
       <color rgba="0.9 0.9 0.9 1"/>
     </material>
-    <joint name="${prefix}_base_joint" type="fixed">
+    <joint name="${prefix}bpearl_base_joint" type="fixed">
       <xacro:insert_block name="origin" />
       <parent link="${parent}"/>
-      <child link="${prefix}_base_link" />
+      <child link="${prefix}bpearl_base_link" />
     </joint>
-    <link name="${prefix}_base_link">
+    <link name="${prefix}bpearl_base_link">
       <visual>
       <!-- origin xyz="0 0 0" rpy="0 0 1.5708"/ -->
@@ -33,10 +33,10 @@
       </inertial>
     </link>
-    <joint name="${prefix}_joint" type="fixed">
-      <parent link="${prefix}_base_link"/>
-      <child link="${prefix}_link" />
+    <joint name="${prefix}bpearl_joint" type="fixed">
+      <parent link="${prefix}bpearl_base_link"/>
+      <child link="${prefix}bpearl_link" />
       <origin xyz="0 0 0.06" rpy="0 0 0"/>
     </joint>
-    <link name="${prefix}_link"/>
+    <link name="${prefix}bpearl_link"/>
   <sensor_rs_bpearl_gazebo range_min="${range_min}" range_max="${range_max}" hfov="${hfov}" samples="${samples}" vfov="${vfov}" lasers="${lasers}" fps="${fps}" gpu="${gpu}"/>
   </xacro:macro>
