Commit message: Fix issue on axis m5525 simulation

File: urdf/axis_m5525.urdf.xacro (robot description, xacro)
@@ -103,4 +103,16 @@
       </inertial>
     </link>
+    <joint name="${prefix}_frame_simulation_joint" type="fixed">
+      <origin xyz="0 0 0" rpy="${M_PI} 0 0"/>
+      <parent link="${prefix}_tilt_link"/>
+      <child link="${prefix}_frame_simulation_link"/>
+    </joint>
+    <link name="${prefix}_frame_simulation_link">
+      <inertial>
+        <mass value="0.1"/>
+        <origin xyz="0 0 0"/>
+        <xacro:solid_cuboid_inertia m="0.1" w="0.11" h="0.11" d="0.1" />
+      </inertial>
+    </link>
     <!-- Optical frame -->
     <joint name="${prefix}_optical_joint" type="fixed">
@@ -116,5 +128,18 @@
       </inertial>
     </link>
-    <gazebo reference="${prefix}_base_link">
+    <!-- For simulation, the link has to be inverted -->
+    <joint name="${prefix}_optical_simulation_joint" type="fixed">
+      <origin xyz="0 0 0" rpy="${-M_PI/2} 0 ${-M_PI/2}"/>
+      <parent link="${prefix}_frame_simulation_link"/>
+      <child link="${prefix}_optical_frame_simulation_link"/>
+    </joint>
+    <link name="${prefix}_optical_frame_simulation_link">
+      <inertial>
+        <mass value="0.1"/>
+        <origin xyz="0 0 0"/>
+        <xacro:solid_cuboid_inertia m="0.1" w="0.11" h="0.11" d="0.1" />
+      </inertial>
+    </link>
+    <gazebo reference="${prefix}_base_simulation_link">
       <material>Gazebo/DarkGrey</material>
     </gazebo>
@@ -123,5 +148,5 @@
   </xacro:macro>
 	<xacro:macro name="sensor_axis_m5525_gazebo">
-		<gazebo reference="${prefix}_frame_link"> <!-- the image will be generated from this (${name}_frame) point of view, with the front being the X axis -->
+		<gazebo reference="${prefix}_frame_simulation_link"> <!-- the image will be generated from this (${name}_frame) point of view, with the front being the X axis -->
 			<sensor type="camera" name="${prefix}_sensor">
 				<update_rate>30.0</update_rate>
@@ -144,5 +169,5 @@
 					<imageTopicName>image_raw</imageTopicName>
 					<cameraInfoTopicName>camera_info</cameraInfoTopicName>
-					<frameName>${prefix}_optical_frame_link</frameName>
+					<frameName>${prefix}_optical_frame_simulation_link</frameName>
 					<!-- this is just which name the Image msg will have, it does not affect the simulation.
 					     However must be set to the optical_frame,  -->

Commit message: Fix axis m5525 TF

File: urdf/axis_m5525.urdf.xacro (robot description, xacro)
@@ -68,5 +68,5 @@
     <joint name="${prefix}_tilt_joint" type="revolute">
       <axis xyz="0 -1 0"/>
-      <origin xyz="0.0 0.0 0.0" rpy="0 ${-PI/2} 0"/>
+      <origin xyz="0.0 0.0 0.0" rpy="0 ${PI/2} 0"/>
       <parent link="${prefix}_pan_link"/>
       <child link="${prefix}_tilt_link"/>
@@ -103,16 +103,4 @@
       </inertial>
     </link>
-    <joint name="${prefix}_frame_simulation_joint" type="fixed">
-      <origin xyz="0 0 0" rpy="${M_PI} 0 0"/>
-      <parent link="${prefix}_tilt_link"/>
-      <child link="${prefix}_frame_simulation_link"/>
-    </joint>
-    <link name="${prefix}_frame_simulation_link">
-      <inertial>
-        <mass value="0.1"/>
-        <origin xyz="0 0 0"/>
-        <xacro:solid_cuboid_inertia m="0.1" w="0.11" h="0.11" d="0.1" />
-      </inertial>
-    </link>
     <!-- Optical frame -->
     <joint name="${prefix}_optical_joint" type="fixed">
@@ -128,18 +116,5 @@
       </inertial>
     </link>
-    <!-- For simulation, the link has to be inverted -->
-    <joint name="${prefix}_optical_simulation_joint" type="fixed">
-      <origin xyz="0 0 0" rpy="${-M_PI/2} 0 ${-M_PI/2}"/>
-      <parent link="${prefix}_frame_simulation_link"/>
-      <child link="${prefix}_optical_frame_simulation_link"/>
-    </joint>
-    <link name="${prefix}_optical_frame_simulation_link">
-      <inertial>
-        <mass value="0.1"/>
-        <origin xyz="0 0 0"/>
-        <xacro:solid_cuboid_inertia m="0.1" w="0.11" h="0.11" d="0.1" />
-      </inertial>
-    </link>
-    <gazebo reference="${prefix}_base_simulation_link">
+    <gazebo reference="${prefix}_base_link">
       <material>Gazebo/DarkGrey</material>
     </gazebo>
@@ -148,5 +123,5 @@
   </xacro:macro>
 	<xacro:macro name="sensor_axis_m5525_gazebo">
-		<gazebo reference="${prefix}_frame_simulation_link"> <!-- the image will be generated from this (${name}_frame) point of view, with the front being the X axis -->
+		<gazebo reference="${prefix}_frame_link"> <!-- the image will be generated from this (${name}_frame) point of view, with the front being the X axis -->
 			<sensor type="camera" name="${prefix}_sensor">
 				<update_rate>30.0</update_rate>
@@ -169,5 +144,5 @@
 					<imageTopicName>image_raw</imageTopicName>
 					<cameraInfoTopicName>camera_info</cameraInfoTopicName>
-					<frameName>${prefix}_optical_frame_simulation_link</frameName>
+					<frameName>${prefix}_optical_frame_link</frameName>
 					<!-- this is just which name the Image msg will have, it does not affect the simulation.
 					     However must be set to the optical_frame,  -->
