Commit message: add params to modify imu properties

File: urdf/imu.urdf.xacro (robot description, xacro)
@@ -1,5 +1,5 @@
 <?xml version="1.0"?>
 <robot name="sensor_imu" xmlns:xacro="http://wiki.ros.org/xacro">
-  <xacro:macro name="sensor_imu" params="prefix ns:='' parent *origin">
+  <xacro:macro name="sensor_imu" params="prefix ns:='' parent *origin topic_name:='imu/data' rate:='100' gaussian_noise:='0.01' xyzoffset:='0 0 0' rpyoffset:='0 0 0'">
 	  <joint name="${prefix}_joint" type="fixed">
 	      <axis xyz="1 0 0"/>
@@ -41,14 +41,14 @@
     <sensor name="${prefix}_imu_sensor" type="imu">
       <always_on>true</always_on>
-      <update_rate>100</update_rate>
+      <update_rate>${rate}</update_rate>
       <visualize>true</visualize>
       <topic>__default_topic__</topic>
       <plugin filename="libgazebo_ros_imu_sensor.so" name="${prefix}_imu_plugin">
-        <topicName>imu/data</topicName>
+        <topicName>${topic_name}</topicName>
 		<bodyName>${prefix}_link</bodyName>
-        <updateRateHZ>100.0</updateRateHZ>
-        <gaussianNoise>0.0</gaussianNoise>
-        <xyzOffset>0 0 0</xyzOffset>
-        <rpyOffset>0 0 0</rpyOffset>
+        <updateRateHZ>${rate}</updateRateHZ>
+        <gaussianNoise>${gaussian_noise}</gaussianNoise>
+        <xyzOffset>${xyzoffset}</xyzOffset>
+        <rpyOffset>${rpyoffset}</rpyOffset>
 		<frameName>${prefix}_link</frameName>
       </plugin>
